Commit message: update gazebo from classic to harmonic

File: ros2_SimRealRobotControl/packages/ur5/ros2srrc_ur5_gazebo/urdf/cam_on_base.xacro (robot description, xacro)
@@ -11,5 +11,4 @@
         <visual>
             <geometry>
-                <!-- <box size="0.01 0.03 0.03" /> -->
                 <mesh filename="file://$(find ros2srrc_ur5_gazebo)/meshes/kinetic.stl"/>
             </geometry>
@@ -33,24 +32,23 @@
         <parent link="base_camera_link"/>
         <child link="base_camera_optical_link"/>
-        <origin xyz="0 0 0" rpy="-1.57 0 -1.57" />
+        <origin xyz="0 0 0" rpy="0 0 0" />
     </joint>
+    <!-- CHANGED: replaced libgazebo_ros_camera.so (Classic) with native Gazebo Harmonic depth sensor -->
+    <!-- Topics are bridged to ROS 2 via ros_gz_bridge in the launch file:                          -->
+    <!--   /base_camera/depth/image_raw  -> sensor_msgs/msg/Image                                   -->
+    <!--   /base_camera/color/image_raw  -> sensor_msgs/msg/Image                                   -->
+    <!--   /base_camera/points           -> sensor_msgs/msg/PointCloud2                             -->
     <gazebo reference="base_camera_link">
-        <visual>
-            <geometry>
-                <mesh>
-                    <mesh filename="file://$(find ros2srrc_ur5_gazebo)/meshes/kinetic.stl"/>
-                </mesh>
-            </geometry>
-            <material>Gazebo/Red</material>
-        </visual>
-        <!-- <material>Gazebo/Red</material> -->
-        <sensor name="base_camera" type="depth">
-            <pose> 0 0 0 0 0 0 </pose>
+        <sensor name="base_camera" type="rgbd_camera">
+            <pose>0 0 0 0 0 0</pose>
+            <always_on>1</always_on>
+            <update_rate>10</update_rate>
             <visualize>true</visualize>
-            <update_rate>10</update_rate>
+            <topic>base_camera</topic>
+            <gz_frame_id>base_camera_optical_link</gz_frame_id>
             <camera>
                 <horizontal_fov>1.047</horizontal_fov>
                 <image>
-                    <format>B8G8R8</format>
+                    <format>R8G8B8</format>
                     <width>640</width>
                     <height>480</height>
@@ -61,16 +59,5 @@
                 </clip>
             </camera>
-            <plugin name="base_camera_controller" filename="libgazebo_ros_camera.so" >
-                <frame_name>base_camera_optical_link</frame_name>
-            </plugin>
         </sensor>
     </gazebo>
-    <gazebo reference="base_camera_link">
-        <visual>
-            <geometry>
-                <mesh filename="file://$(find ros2srrc_ur5_gazebo)/meshes/kinetic.stl"/>
-            </geometry>
-            <material>Gazebo/Red</material>
-        </visual>
-    </gazebo>
 </robot>

File: ros2_SimRealRobotControl/packages/ur5/ros2srrc_ur5_gazebo/urdf/cam_on_hand.xacro (robot description, xacro)
@@ -11,5 +11,4 @@
         <visual>
             <geometry>
-                <!-- <box size="0.01 0.03 0.03" /> -->
                 <mesh filename="file://$(find ros2srrc_ur5_gazebo)/meshes/kinetic.stl"/>
             </geometry>
@@ -35,21 +34,21 @@
         <origin xyz="0 0 0" rpy="-1.57 0 -1.57" />
     </joint>
+    <!-- CHANGED: replaced libgazebo_ros_camera.so (Classic) with native Gazebo Harmonic depth sensor -->
+    <!-- Topics are bridged to ROS 2 via ros_gz_bridge in the launch file:                          -->
+    <!--   /hand_camera/depth/image_raw  -> sensor_msgs/msg/Image                                   -->
+    <!--   /hand_camera/color/image_raw  -> sensor_msgs/msg/Image                                   -->
+    <!--   /hand_camera/points           -> sensor_msgs/msg/PointCloud2                             -->
     <gazebo reference="hand_camera_link">
-        <visual>
-            <geometry>
-                <mesh>
-                    <mesh filename="file://$(find ros2srrc_ur5_gazebo)/meshes/kinetic.stl"/>
-                </mesh>
-            </geometry>
-            <material>Gazebo/Red</material>
-        </visual>
-        <sensor name="hand_camera" type="depth">
-            <pose> 0 0 0 0 0 0 </pose>
+        <sensor name="hand_camera" type="rgbd_camera">
+            <pose>0 0 0 0 0 0</pose>
+            <always_on>1</always_on>
+            <update_rate>10</update_rate>
             <visualize>true</visualize>
-            <update_rate>10</update_rate>
+            <topic>hand_camera</topic>
+            <gz_frame_id>hand_camera_optical_link</gz_frame_id>
             <camera>
                 <horizontal_fov>1.047</horizontal_fov>
                 <image>
-                    <format>B8G8R8</format>
+                    <format>R8G8B8</format>
                     <width>640</width>
                     <height>480</height>
@@ -60,16 +59,5 @@
                 </clip>
             </camera>
-            <plugin name="hand_camera_controller" filename="libgazebo_ros_camera.so" >
-                <frame_name>hand_camera_optical_link</frame_name>
-            </plugin>
         </sensor>
     </gazebo>
-    <gazebo reference="hand_camera_link">
-        <visual>
-            <geometry>
-                <mesh filename="file://$(find ros2srrc_ur5_gazebo)/meshes/kinetic.stl"/>
-            </geometry>
-            <material>Gazebo/Red</material>
-        </visual>
-    </gazebo>
 </robot>

File: ros2_SimRealRobotControl/packages/ur5/ros2srrc_ur5_gazebo/urdf/ur5_robotiq_2f85_with_cams.urdf.xacro (robot description, xacro)
@@ -24,7 +24,4 @@
 #                                                                                       #
 # ===================================== COPYRIGHT ===================================== #
-# ======= CITE OUR WORK ======= #
-# You can cite our work with the following statement:
-# IFRA-Cranfield (2023) ROS 2 Sim-to-Real Robot Control. URL: https://github.com/IFRA-Cranfield/ros2_SimRealRobotControl.
 -->
 <robot name="ur5" xmlns:xacro="http://ros.org/wiki/xacro">
@@ -69,9 +66,10 @@
     parent_link="tool0"
   />
-  <!-- Load ROS 2 Gazebo Plugin -->
+  <!-- Load ROS 2 Gazebo Harmonic Plugin -->
+  <!-- CHANGED: libgazebo_ros2_control.so (Classic) -> gz_ros2_control-system (Harmonic) -->
   <xacro:unless value="${bringup}">
     <gazebo>
-      <plugin filename="libgazebo_ros2_control.so" name="gazebo_ros2_control">
-        <robot_sim_type>gazebo_ros2_control/GazeboSystem</robot_sim_type>
+      <plugin filename="gz_ros2_control-system"
+              name="gz_ros2_control::GazeboSimROS2ControlPlugin">
         <!-- UR5 Controller -->
         <parameters>$(find ros2srrc_robots)/ur5/config/controller.yaml</parameters>

File: ros2_SimRealRobotControl/ros2srrc_robots/ur5/urdf/ur5_ros2control.xacro (robot description, xacro)
@@ -10,9 +10,4 @@
 #  You may not use this file except in compliance with the License.                     #
 #  You may obtain a copy of the License at: http://www.apache.org/licenses/LICENSE-2.0  #
-#                                                                                       #
-#  Unless required by applicable law or agreed to in writing, software distributed      #
-#  under the License is distributed on an "as-is" basis, without warranties or          #
-#  conditions of any kind, either express or implied. See the License for the specific  #
-#  language governing permissions and limitations under the License.                    #
 #                                                                                       #
 #  IFRA Group - Cranfield University                                                    #
@@ -24,33 +19,4 @@
 #                                                                                       #
 # ===================================== COPYRIGHT ===================================== #
-# ===================================== COPYRIGHT ===================================== #
-#                                                                                       #
-#  Some of the information used to build the ROS2 UR5-Robot .urdf files in this ROS2    #
-#  repository has been taken from the following resources:                              #
-#       - Universal Robots ROS2 Description:                                            #
-#         https://github.com/UniversalRobots/Universal_Robots_ROS2_Description          #
-#       - Universal Robots ROS2 Gazebo Simulation:                                      #
-#         https://github.com/UniversalRobots/Universal_Robots_ROS2_Gazebo_Simulation    #
-#                                                                                       #
-#  AUTHORS:                                                                             #
-#       - ROS-Industrial - https://rosindustrial.org                                    #
-#       - Universal Robots - https://github.com/UniversalRobots                         #
-#       - Nadia Hammoudeh Garcia, Kelsey Hawkins, G.A. vd. Hoorn, Lovro Ivanov, Mathias #
-#         Ludtke, Wim Meeussen, Felix Messmer, Miguel Prada Sarasola, Denis Stogl,      #
-#         Andy Zelenak, Marvin Grosse Besselmann.                                       #
-#       - Maintainers: Felix Exner (exner@fzi.de), Tristan Schnell (schnell@fzi.de),    #
-#         Lovro Ivanov (lovro.ivanov@gmail.com), Denis Stogl (denis@stoglrobotics.de).  #
-#                                                                                       #
-#  Copyright (c) 2021, Universal Robots A/S                                             #
-#  (ORIGINAL LICENSE) -> Licensed under the BSD 3-Clause License.                       #
-#                                                                                       #
-#  CHANGES MADE:                                                                        #
-#  Robot information/specifications have been taken, and the code has been modified and #
-#  re-organised in accordance with the ros2_SimRealRobotControl standards.              #
-#                                                                                       #
-# ===================================== COPYRIGHT ===================================== #
-# ======= CITE OUR WORK ======= #
-# You can cite our work with the following statement:
-# IFRA-Cranfield (2023) ROS 2 Sim-to-Real Robot Control. URL: https://github.com/IFRA-Cranfield/ros2_SimRealRobotControl.
 -->
 <robot xmlns:xacro="http://www.ros.org/wiki/xacro">
@@ -110,8 +76,9 @@
     <!-- Load ROS2_CONTROL: -->
     <ros2_control name="${name}" type="system">
-      <!-- A. GAZEBO SIMULATION: -->
+      <!-- A. GAZEBO HARMONIC SIMULATION: -->
+      <!-- CHANGED: gazebo_ros2_control/GazeboSystem (Classic) -> gz_ros2_control/GazeboSimSystem (Harmonic) -->
       <xacro:unless value="${bringup}">
         <hardware>
-          <plugin>gazebo_ros2_control/GazeboSystem</plugin>
+          <plugin>gz_ros2_control/GazeboSimSystem</plugin>
         </hardware>
       </xacro:unless>
@@ -282,24 +249,24 @@
         </xacro:if>
       </xacro:unless>
-      <!-- DMM: SOLO PARA EJE YAMAHA, PENDIENTE DE RELOCALIZAR CORRECTAMENTE EN ARCHIVO APARTE QUE CARGUE SOLO SI HAY EJE -->
-     <joint name="yamaha_joint">
-      <command_interface name="position">
-        <param name="min">-0.9</param>
-        <param name="max">0.9</param>
-      </command_interface>
-      <command_interface name="velocity">
-        <param name="min">0.1</param>
-        <param name="max">1.0</param>
-      </command_interface>
-      <state_interface name="position">
-        <param name="initial_value">0.0</param>
-      </state_interface>
-      <state_interface name="velocity">
-        <param name="initial_value">0.0</param>
-      </state_interface>
-      <state_interface name="effort">
-        <param name="initial_value">0.0</param>
-      </state_interface>
-     </joint>
+      <!-- DMM: SOLO PARA EJE YAMAHA -->
+      <joint name="yamaha_joint">
+        <command_interface name="position">
+          <param name="min">-0.9</param>
+          <param name="max">0.9</param>
+        </command_interface>
+        <command_interface name="velocity">
+          <param name="min">0.1</param>
+          <param name="max">1.0</param>
+        </command_interface>
+        <state_interface name="position">
+          <param name="initial_value">0.0</param>
+        </state_interface>
+        <state_interface name="velocity">
+          <param name="initial_value">0.0</param>
+        </state_interface>
+        <state_interface name="effort">
+          <param name="initial_value">0.0</param>
+        </state_interface>
+      </joint>
     </ros2_control>
     <xacro:unless value="${bringup}">
@@ -322,14 +289,13 @@
         <selfCollide>false</selfCollide>
       </gazebo>
-      <!--YAMAHA AXIS LINKS -->
+      <!-- YAMAHA AXIS LINKS -->
       <gazebo reference="yamaha_axis">
-       <selfCollide>false</selfCollide>
+        <selfCollide>false</selfCollide>
       </gazebo>
       <gazebo reference="robot_stand">
-       <selfCollide>false</selfCollide>
+        <selfCollide>false</selfCollide>
       </gazebo>
       <gazebo reference="end_effector_frame_fixed_joint">
         <preserveFixedJoint>true</preserveFixedJoint>
-        <!-- For compatibility with SDFormat < 4.4 -->
         <disableFixedJointLumping>true</disableFixedJointLumping>
       </gazebo>
